File: UINIO-MCU-RP2040.kicad_pcb (KiCad board)
At the start: 2 copper layers, 0 parts

Commit message: Complete the schematic drawing.
Parts:
- added C1: 1uF, Capacitor_SMD:C_0603_1608Metric, F.Cu at (122.5, 45.6)
- added C10: 0.1uF, Capacitor_SMD:C_0603_1608Metric, F.Cu at (245.9, 90.3)
- added C11: 0.1uF, Capacitor_SMD:C_0603_1608Metric, F.Cu at (249.9, 77.8)
- added C12: 2.2uF, Capacitor_SMD:C_0603_1608Metric, F.Cu at (249.9, 80.3)
- added C13: 0.1uF, Capacitor_SMD:C_0603_1608Metric, F.Cu at (249.9, 82.8)
- added C14: 0.1uF, Capacitor_SMD:C_0603_1608Metric, F.Cu at (249.9, 85.3)
- added C15: 2.2uF, Capacitor_SMD:C_0603_1608Metric, F.Cu at (155.9, 109.9)
- added C16: 1nF, Capacitor_SMD:C_0603_1608Metric, F.Cu at (155.9, 112.4)
- added C2: 1uF, Capacitor_SMD:C_0603_1608Metric, F.Cu at (122.5, 48.1)
- added C3: 0.01uF, Capacitor_SMD:C_0603_1608Metric, F.Cu at (122.5, 50.6)
- added C4: 12pF, Capacitor_SMD:C_0603_1608Metric, F.Cu at (245.9, 77.8)
- added C5: 12pF, Capacitor_SMD:C_0603_1608Metric, F.Cu at (245.9, 80.3)
- added C6: 0.1uF, Capacitor_SMD:C_0603_1608Metric, F.Cu at (245.9, 82.8)
- added C7: 0.1uF, Capacitor_SMD:C_0603_1608Metric, F.Cu at (226.1, 144.6)
- added C8: 0.1uF, Capacitor_SMD:C_0603_1608Metric, F.Cu at (245.9, 85.3)
- added C9: 2.2uF, Capacitor_SMD:C_0603_1608Metric, F.Cu at (245.9, 87.8)
- added D1: 1N5819, Diode_SMD:D_SOD-323F, F.Cu at (122.4, 42.2)
- added D2: LED_Red, LED_SMD:LED_0603_1608Metric, F.Cu at (131.2, 45.7)
- added D3: LED_Blue, LED_SMD:LED_0603_1608Metric, F.Cu at (251.2, 92.9)
- added J1: Conn_01x20_Pin, Connector_PinHeader_2.54mm:PinHeader_1x20_P2.54mm_Vertical, F.Cu at (73.1, 112.6)
- added J2: Conn_01x20_Pin, Connector_PinHeader_2.54mm:PinHeader_1x20_P2.54mm_Vertical, F.Cu at (77.8, 112.6)
- added J3: Conn_01x04_Pin, Connector_PinHeader_2.54mm:PinHeader_1x04_P2.54mm_Vertical, F.Cu at (235.2, 84.4)
- added Q1: DMG1012T, Package_TO_SOT_SMD:SOT-523, F.Cu at (250.8, 95.7)
- added R1: 512R, Resistor_SMD:R_0603_1608Metric, F.Cu at (122.5, 53.2)
- added R10: 200K, Resistor_SMD:R_0603_1608Metric, F.Cu at (253.9, 80.3)
- added R11: 1R, Resistor_SMD:R_0603_1608Metric, F.Cu at (253.9, 82.8)
- added R12: 200R, Resistor_SMD:R_0603_1608Metric, F.Cu at (253.9, 85.3)
- added R13: 1K, Resistor_SMD:R_0603_1608Metric, F.Cu at (253.9, 87.8)
- added R2: 5.1K, Resistor_SMD:R_0603_1608Metric, F.Cu at (199.9, 63.3)
- added R3: 5.1K, Resistor_SMD:R_0603_1608Metric, F.Cu at (199.9, 65.8)
- added R4: 2K, Resistor_SMD:R_0603_1608Metric, F.Cu at (122.5, 55.7)
- added R5: 1.5K, Resistor_SMD:R_0603_1608Metric, F.Cu at (155.9, 114.9)
- added R6: 27K, Resistor_SMD:R_0603_1608Metric, F.Cu at (234.1, 142.1)
- added R7: 27K, Resistor_SMD:R_0603_1608Metric, F.Cu at (249.9, 87.8)
- added R8: 470R, Resistor_SMD:R_0603_1608Metric, F.Cu at (249.9, 90.3)
- added R9: 100K, Resistor_SMD:R_0603_1608Metric, F.Cu at (253.9, 77.8)
- added SW1: ~{RESET}, Uinio:KEY-SMD_4P-L4.2-W3.4-P2.15-LS4.7, F.Cu at (150.6, 111.0)
- added SW2: ~{USB_BOOT}, Uinio:KEY-SMD_4P-L4.2-W3.4-P2.15-LS4.7, F.Cu at (150.6, 115.6)
- added U1: SGM2019-3.3YN5G, Uinio:SOT-23-5_L3.0-W1.7-P0.95-LS2.8-BR, F.Cu at (126.8, 46.6)
- added U2: SPI-25-Flash-WSON8, Package_SON:WSON-8-1EP_6x5mm_P1.27mm_EP3.4x4.3mm, F.Cu at (234.4, 177.4)
- added U3: RP2040, Package_DFN_QFN:QFN-56-1EP_7x7mm_P0.4mm_EP3.2x3.2mm, F.Cu at (260.6, 93.4)
- added USB1: USB_Type_C_16Pin, Uinio:USB-C-SMD_TYPEC-304J-BCP16, F.Cu at (203.3, 56.3)
- added Y1: 12MHz, Crystal:Crystal_SMD_3225-4Pin_3.2x2.5mm, F.Cu at (246.5, 93.8)

Commit message: PCB preliminary layout.
Parts:
- moved U3 160.9 mm to (100.8, 112.6), turned to 45 degrees
- moved U2 160.8 mm to (87.7, 111.6), turned to 90 degrees
- moved USB1 150.2 mm to (63.4, 111.0), turned to -90 degrees
- moved C5 138.7 mm to (112.7, 118.9)
- moved C4 137.3 mm to (112.9, 112.2)
- moved Y1 135.3 mm to (112.9, 115.2), turned to 180 degrees
- moved R2 131.2 mm to (77.0, 109.2)
- moved R3 131.2 mm to (77.0, 111.7)
- moved J3 115.5 mm to (121.9, 106.7)
- moved C11 110.5 mm to (139.4, 78.7)
- moved C12 110.5 mm to (139.4, 81.2)
- moved C13 110.5 mm to (139.4, 83.8)
- moved C14 110.5 mm to (139.4, 86.3)
- moved D3 110.5 mm to (140.7, 93.8)
- moved Q1 110.5 mm to (140.3, 96.7)
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
Commit message: Finish PCB layout.
Parts:
- added HOLE**: Hole-2mm, Uinio:Hole-2mm, F.Cu at (115.1, 112.7)
- added HOLE**: Hole-2mm, Uinio:Hole-2mm, F.Cu at (115.1, 93.6)
- added HOLE**: Hole-2mm, Uinio:Hole-2mm, F.Cu at (170.5, 93.6)
- added HOLE**: Hole-2mm, Uinio:Hole-2mm, F.Cu at (170.5, 112.7)
- C10, C11, C12, C13, C14, C15, C16, C4, C5, C6, C7, C8, C9: footprint Capacitor_SMD:C_0603_1608Metric -> Capacitor_SMD:C_0402_1005Metric
- R10, R11, R13, R5, R6, R7, R8, R9: footprint Resistor_SMD:R_0603_1608Metric -> Resistor_SMD:R_0402_1005Metric
- moved R6 115.9 mm to (124.7, 103.9), turned to 180 degrees
- moved C7 86.2 mm to (153.4, 98.3), turned to 90 degrees
- moved D1 64.8 mm to (124.6, 107.0), turned to 180 degrees
- moved C1 64.6 mm to (130.1, 109.7), turned to 180 degrees
- moved U1 60.6 mm to (130.1, 107.0), turned to -90 degrees
- moved R1 56.6 mm to (124.7, 109.7), turned to 180 degrees
- moved C2 56.6 mm to (130.1, 104.2), turned to 180 degrees
- moved USB1 53.4 mm to (116.3, 103.1)
- moved C3 52.6 mm to (130.1, 102.7)
- moved D2 51.9 mm to (130.1, 97.6)
- moved J3 51.0 mm to (172.4, 99.3)
- moved U2 50.8 mm to (138.3, 107.2)
- moved C5 50.2 mm to (157.8, 96.9)
- moved R3 49.2 mm to (124.7, 99.5), turned to 180 degrees
- moved R2 49.0 mm to (124.7, 97.5), turned to 180 degrees
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Connections:
- C1 pad 2: Net-(D1-K) -> /VDD_5V
- D1 pad 1: Net-(D1-K) -> /VDD_5V
- D1 pad 2: /VDD_5V -> /USB_5V
- R1 pad 1: Net-(D1-K) -> /VDD_5V
- R6 pad 1: Net-(U3-USB_DP) -> /USB_Data+
- R6 pad 2: /USB_Data+ -> Net-(USB1-DP1)
- R7 pad 1: Net-(U3-USB_DM) -> /USB_Data-
- R7 pad 2: /USB_Data- -> Net-(USB1-DN1)
- U1 pad 1: Net-(D1-K) -> /VDD_5V
- U3 pad 46: Net-(U3-USB_DM) -> /USB_Data-
- U3 pad 47: Net-(U3-USB_DP) -> /USB_Data+
- USB1 pad A4B9: /VDD_5V -> /USB_5V
- USB1 pad A6: /USB_Data+ -> Net-(USB1-DP1)
- USB1 pad A7: /USB_Data- -> Net-(USB1-DN1)
- USB1 pad B4A9: /VDD_5V -> /USB_5V
- USB1 pad B6: /USB_Data+ -> Net-(USB1-DP1)
- USB1 pad B7: /USB_Data- -> Net-(USB1-DN1)
Other:
- board outline added: 61.9 x 25.4 mm
- board text added: "3V3"
- board text added: "5V"
- board text added: "BOOT"
- board text added: "EN"
- board text added: "G0"
- board text added: "G1"
- board text added: "G10"
- board text added: "G11"
- board text added: "G12"
- board text added: "G13"
- board text added: "G14"
- board text added: "G15"
- board text added: "G16"
- board text added: "G17"
- board text added: "G18"
- board text added: "G19"
- board text added: "G2"
- board text added: "G20"
- board text added: "G21"
- board text added: "G22"
- board text added: "G23"
- board text added: "G24"
- board text added: "G26"
- board text added: "G27"
- board text added: "G28"
- board text added: "G4"
- board text added: "G5"
- board text added: "G6"
- board text added: "G7"
- board text added: "G8"
- board text added: "G9"
- board text added: "GND"
- board text added: "REST"
- board text added: "RP2040"
- board text added: "RUN"
- board text added: "Raspberry Pi"
- board text added: "SCLK"
- board text added: "SWD"
- board text added: "UinIO.com"
- board text added: "VREF"

Commit message: Complete PCB wiring.
Parts:
- added C17: 0.1uF, Capacitor_SMD:C_0402_1005Metric, F.Cu at (157.2, 95.6)
- D1: footprint Diode_SMD:D_SOD-323F -> Diode_SMD:D_SOD-123
- moved R13 5.92 mm to (166.9, 101.8)
- moved SW2 5.92 mm to (168.1, 104.3)
- moved SW1 5.92 mm to (168.1, 96.6)
- moved C13 5.92 mm to (169.3, 99.0)
- moved C14 5.92 mm to (169.3, 101.8)
- moved C15 5.73 mm to (143.8, 97.0)
- moved C11 5.55 mm to (146.7, 103.5)
- moved C7 5.36 mm to (157.2, 94.5), turned to 0 degrees
- moved D1 5.22 mm to (129.0, 104.2)
- moved U1 5.01 mm to (134.3, 104.3)
- moved R11 4.93 mm to (141.4, 98.2)
- moved Q1 4.93 mm to (161.6, 104.4)
- moved C4 4.91 mm to (161.8, 99.3)
- moved R12 4.89 mm to (141.0, 96.6), turned to 180 degrees
- moved C12 4.88 mm to (143.8, 95.8)
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Connections:
- J1 pad 2: /VDD_3.3V -> /VDD_5V
- J2 pad 1: /VDD_5V -> GND
- J2 pad 11: /RUN -> /GPIO22
- J2 pad 12: /GPIO22 -> /GPIO21
- J2 pad 13: /GPIO21 -> /GPIO20
- J2 pad 14: /GPIO20 -> /GPIO19
- J2 pad 15: /GPIO19 -> /GPIO18
- J2 pad 16: /GPIO18 -> /GPIO17
- J2 pad 17: /GPIO17 -> /GPIO16
- J2 pad 18: /GPIO16 -> /RUN
- J2 pad 2: GND -> /VDD_3.3V
- J2 pad 3: /VDD_3.3V -> GND
- J3 pad 1: GND -> /VDD_3.3V
- J3 pad 4: /VDD_3.3V -> GND
- U3 pad 24: Net-(J3-Pin_2) -> Net-(J3-Pin_3)
- U3 pad 25: Net-(J3-Pin_3) -> Net-(J3-Pin_2)
Routing:
- net /VDD_3.3V: track 0.00 -> 163.3 mm, vias 0 -> 10
- net /VDD_5V: track 0.00 -> 50.1 mm, vias 0 -> 2
- net /Boot_Select: track 0.00 -> 47.6 mm, vias 0 -> 2
- net GND: track 0.00 -> 41.3 mm, vias 0 -> 47
- net /RUN: track 0.00 -> 31.6 mm, vias 0 -> 1
- net /LDO_EN: track 0.00 -> 31.0 mm, vias 0 -> 1
- net /GPIO0: track 0.00 -> 29.6 mm
- net Net-(J3-Pin_3): track 0.00 -> 28.9 mm
- net /GPIO1: track 0.00 -> 27.6 mm
- net Net-(J3-Pin_2): track 0.00 -> 27.1 mm
- net /GPIO2: track 0.00 -> 25.7 mm
- net +1V1: track 0.00 -> 24.9 mm
- net /GPIO3: track 0.00 -> 23.7 mm
- net /USB_Data+: track 0.00 -> 22.4 mm
- net /USB_Data-: track 0.00 -> 22.1 mm
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- added copper zone on B.Cu, net GND
- added copper zone on F.Cu, net GND
Other:
- outline, holes or cut-outs redrawn
- board text added: "UINIO-MCU-RP2040"
- board text added: "Version 1.0.0"
