File: UINIO-MCU-RP2040.kicad_pcb (KiCad board)
At the start: 2 copper layers, 61.9 x 25.4 mm, 47 parts, among them J1 Conn_01x20_Pin, J2 Conn_01x20_Pin, J3 Conn_01x04_Pin, Q1 DMG1012T, SW1 ~{RESET}, SW2 ~{USB_BOOT}, U1 SGM2019-3.3YN5G, U2 SPI-25-Flash-WSON8, U3 RP2040, Y1 12MHz

Commit message: Release UINIO-MCU-RP2040 version 2.2.0.
Routing:
- net /VDD_3.3V: track 166.3 -> 168.5 mm
- net /VDD_5V: track 50.1 -> 48.3 mm
- net /Boot_Select: track 50.1 -> 48.9 mm
- net /RUN: track 31.7 -> 31.0 mm
- net GND: track 31.4 -> 31.8 mm, vias 41 -> 85
Other:
- board text added: "Version 2.2.0"
- board text removed: "Version 2.0.0"

Commit message: Release UINIO-MCU-RP2040 version 2.2.0.
Routing:
- net /USB_5V: track 11.5 -> 13.6 mm
- net GND: vias 85 -> 68
