File: UINIO-MCU-RP2040.kicad_pcb (KiCad board)
At the start: 2 copper layers, 61.9 x 25.4 mm, 47 parts, among them J1 Conn_01x20_Pin, J2 Conn_01x20_Pin, J3 Conn_01x04_Pin, Q1 DMG1012T, SW1 ~{RESET}, SW2 ~{USB_BOOT}, U1 SGM2019-3.3YN5G, U2 SPI-25-Flash-WSON8, U3 RP2040, Y1 12MHz

Commit message: Release UINIO-MCU-RP2040 version 3.0.0.
Other:
- board text added: "Version 3.0.0"
- board text removed: "Version 2.2.0"

Commit message: update
Parts:
- added D4: LESD5D5.0CT1G, Diode_SMD:D_SOD-523, F.Cu at (128.7, 99.1)
- added D5: LESD5D5.0CT1G, Diode_SMD:D_SOD-523, F.Cu at (128.7, 101.6)
- added F1: 60V 1A, Fuse:Fuse_1206_3216Metric, F.Cu at (129.0, 106.6)
- added HOLE**: Hole-2mm, Uinio:Hole-2mm, F.Cu at (187.5, 92.3)
- added HOLE**: Hole-2mm, Uinio:Hole-2mm, F.Cu at (191.3, 92.5)
- added HOLE**: Hole-2mm, Uinio:Hole-2mm, F.Cu at (188.4, 87.5)
- added HOLE**: Hole-2mm, Uinio:Hole-2mm, F.Cu at (182.6, 88.5)
- D1: value 1N5819 -> 1N4007; footprint Diode_SMD:D_SOD-123 -> Diode_SMD:Nexperia_CFP3_SOD-123W
- moved R1 13.6 mm to (128.6, 93.4)
- moved R6 2.13 mm to (130.8, 100.9)
- moved R7 2.13 mm to (130.8, 99.8)
- moved HOLE** 1.28 mm to (174.5, 89.5)
- moved HOLE** 1.28 mm to (119.0, 89.5)
- moved J2 1.28 mm to (122.6, 87.7)
- moved HOLE** 1.27 mm to (119.0, 111.2)
- moved HOLE** 1.26 mm to (174.5, 111.2)
- moved J1 1.26 mm to (122.6, 113.0)
- moved C3 0.50 mm to (134.6, 100.0)
- moved C1 0.49 mm to (134.6, 107.0)
- moved C2 0.49 mm to (134.6, 101.4)
- moved D2 0.49 mm to (134.6, 94.8)
- moved R4 0.49 mm to (134.6, 96.7)
- moved U1 0.49 mm to (134.8, 104.3)
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Connections:
- C1 pad 2: /VDD_5V -> /USB_5V
- C2 pad 2: /VDD_3.3V -> Net-(U1-OUT)
- D1 pad 1: /VDD_5V -> /VDD_3.3V
- D1 pad 2: /USB_5V -> GND
- J1 pad 2: /VDD_5V -> /USB_5V
- R1 pad 1: /VDD_5V -> /USB_5V
- R10 pad 2: /VDD_5V -> /USB_5V
- R4 pad 2: /VDD_3.3V -> Net-(U1-OUT)
- U1 pad 1: /VDD_5V -> /USB_5V
- U1 pad 5: /VDD_3.3V -> Net-(U1-OUT)
Routing:
- net (no net): track 0.00 -> 49.7 mm
- net /VDD_5V: track 48.3 -> 0.00 mm, vias 2 -> 0
- net /GPIO28_ADC2: track 20.9 -> 0.00 mm
- net /GPIO27_ADC1: track 18.4 -> 0.00 mm
- net /GPIO26_ADC0: track 15.8 -> 0.00 mm
- net /GPIO16: track 13.7 -> 0.00 mm
- net /GPIO24: track 13.2 -> 0.00 mm
- net /GPIO17: track 11.2 -> 0.00 mm
- net /GPIO23: track 10.7 -> 0.00 mm
- net /GPIO18: track 9.72 -> 0.00 mm
- net /GPIO19: track 9.48 -> 0.00 mm
- net /GPIO22: track 9.47 -> 0.00 mm
- net /GPIO20: track 8.79 -> 0.00 mm
- net /GPIO21: track 8.09 -> 0.00 mm
- net GND: track 31.8 -> 26.7 mm, vias 68 -> 54
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Other:
- board size 61.9 x 25.4 mm -> 62 x 27.9 mm

Commit message: Release UINIO-MCU-RP2040 version 3.2.0.
Parts:
- removed the HOLE** at (119.0, 111.2)
- removed the HOLE** at (119.0, 89.5)
- removed the HOLE** at (174.5, 89.5)
- removed the HOLE** at (174.5, 111.2)
- moved HOLE** 74.7 mm to (119.0, 111.2)
- moved HOLE** 69.4 mm to (119.0, 89.5)
- moved HOLE** 22.9 mm to (174.5, 111.2)
- moved HOLE** 8.14 mm to (174.5, 89.5)
- moved D1 2.13 mm to (128.2, 106.4), turned to -90 degrees
- moved R4 1.90 mm to (134.6, 94.8)
- moved C3 1.66 mm to (135.7, 101.2), turned to -90 degrees
- moved F1 1.64 mm to (130.7, 106.4), turned to -90 degrees
- moved D2 1.36 mm to (134.6, 93.4)
- moved C1 0.95 mm to (134.6, 107.9)
- moved C2 0.81 mm to (133.8, 101.2), turned to -90 degrees
- moved U1 0.62 mm to (134.8, 104.9)
- moved C4 0.38 mm to (161.8, 99.7)
- moved Y1 0.38 mm to (161.0, 97.1)
- moved C5 0.38 mm to (161.8, 94.5)
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Connections:
- R4 pad 2: Net-(U1-OUT) -> /VDD_3.3V
Routing:
- net /USB_5V: track 13.9 -> 74.6 mm
- net (no net): track 49.7 -> 0.00 mm
- net /GPIO28_ADC2: track 0.00 -> 19.5 mm
- net /VDD_3.3V: track 171.6 -> 189.4 mm, vias 10 -> 12
- net /GPIO27_ADC1: track 0.00 -> 17.0 mm
- net /GPIO26_ADC0: track 0.00 -> 14.6 mm
- net /GPIO16: track 0.00 -> 14.0 mm
- net /GPIO24: track 0.00 -> 13.2 mm
- net /GPIO23: track 0.00 -> 12.0 mm
- net /GPIO17: track 0.00 -> 11.6 mm
- net /GPIO18: track 0.00 -> 11.0 mm
- net /GPIO22: track 0.00 -> 10.8 mm
- net /GPIO19: track 0.00 -> 10.6 mm
- net GND: track 26.7 -> 36.8 mm, vias 54 -> 56
- net /GPIO20: track 0.00 -> 9.99 mm
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Other:
- board text added: "Version 3.2.0"
- board text removed: "Version 3.0.0"

Commit message: Release UINIO-MCU-RP2040 version 3.2.0.
Parts:
- moved R11 2.00 mm to (140.1, 96.7), turned to -90 degrees
- moved C15 1.84 mm to (141.9, 96.7), turned to 90 degrees
- moved R12 1.79 mm to (141.0, 94.8)
- moved D3 1.36 mm to (141.0, 93.4)
Routing:
- net GND: track 36.8 -> 51.5 mm, vias 56 -> 74
- net /VDD_3.3V: track 189.4 -> 197.2 mm, vias 12 -> 11
- net /ADC_AVDD: track 8.32 -> 9.57 mm
- net /ADC_VREF: track 13.8 -> 12.7 mm
- net Net-(D3-A): track 1.16 -> 1.88 mm
- net /LDO_EN: track 24.0 -> 23.3 mm

Commit message: Release UINIO-MCU-RP2040 version 5.0.0.
Routing:
- net /VDD_3.3V: track 197.2 -> 195.4 mm
